File: solderclub.kicad_pcb (KiCad board)
At the start: 2 copper layers, 98.2 x 123.9 mm, 21 parts, among them Q1 NPN, Q2 NPN, Q3 NPN

Commit message: Update solderclub.kicad_pcb
Parts:
- moved G*** 9.93 mm to (206.2, 143.7)
- moved G*** 6.67 mm to (143.5, 140.0)
- moved G*** 4.53 mm to (197.0, 141.5)
- moved G*** 1.58 mm to (190.5, 96.5)
Other:
- board size 98.2 x 123.9 mm -> 93.5 x 100 mm
